Commit message: Works with a single axis on Somanet Node. TODO: Homing.

File: hamal_description/urdf/hamal_simple.urdf.xacro (robot description, xacro)
@@ -73,5 +73,5 @@
   </joint>
   <link
-    name="right_wheel_joint">
+    name="rw_link">
     <visual>
       <origin
@@ -88,5 +88,5 @@
   </link>
   <joint
-    name="rw_joint"
+    name="right_wheel_joint"
     type="continuous">
       <origin

File: hamal_description/urdf/moobot.urdf.xacro (robot description, xacro)
@@ -1,6 +1,6 @@
 <?xml version="1.0"?>
 <robot name="hamal" xmlns:xacro="http://ros.org/wiki/xacro">
-  <xacro:include filename="$(find hamal_description)/urdf/common_properties.xacro" />
-  <xacro:include filename="$(find hamal_description)/urdf/moobot.gazebo.xacro" />
+  <!-- <xacro:include filename="$(find hamal_description)/urdf/common_properties.xacro" />
+  <xacro:include filename="$(find hamal_description)/urdf/moobot.gazebo.xacro" /> -->
   <!-- AGV Base -->
   <link name="base_link">
@@ -291,5 +291,5 @@
   </link>
   <!-- Rear Right Mid Wheel Joint  -->
-  <joint name="RRM_wheel_joint" type="continuous">
+  <joint name="right_wheel_joint" type="continuous">
     <parent link="rear_right_buggy_link" />
     <child link="RRM_wheel_link" />
@@ -451,5 +451,5 @@
   </link>
   <!-- Rear Left Mid Wheel Joint  -->
-  <joint name="RLM_wheel_joint" type="continuous">
+  <joint name="left_wheel_joint" type="continuous">
     <parent link="rear_left_buggy_link" />
     <child link="RLM_wheel_link" />

Commit message: Fixed issue while getting current position from PosVelAcc joint handle.

File: hamal_description/urdf/hamal_simple.urdf.xacro (robot description, xacro)
@@ -102,4 +102,30 @@
       k_velocity="0" />
   </joint>
+  <link
+    name="lifter_link">
+    <visual>
+      <origin
+        xyz="0 0 0"
+        rpy="1.5707963267949 0 0" />
+      <geometry>
+        <mesh
+          filename="package://hamal_description/mesh/wheel.stl" />
+      </geometry>
+      <material
+        name="red">
+      </material>
+    </visual>
+  </link>
+  <joint
+    name="lifter_joint"
+    type="continuous">
+      <origin
+      xyz="0 0 0"
+      rpy="0 0 0" />
+    <parent
+      link="base_link" />
+    <child
+      link="lifter_link" />
+  </joint>
   <!-- <joint name="hokuyo_joint" type="fixed">
      <origin xyz="0.35 -0.28 0.09" rpy="0.0 0.0 -0.785"/>

Commit message: Updated the localization package to have the IMU driver, filter options and the EKF filter.

File: hamal_description/urdf/hamal_simple.urdf.xacro (robot description, xacro)
@@ -12,5 +12,5 @@
       <geometry>
         <mesh
-          filename="package://hamal_description/mesh/logos_maxi_base.stl" />
+          filename="package://hamal_description/mesh/logos_maxi_base.stl" scale="0.001 0.001 0.001"/>
       </geometry>
       <collision>
@@ -20,5 +20,5 @@
       <geometry>
         <mesh
-          filename="package://hamal_description/mesh/logos_maxi_base.stl" />
+          filename="package://hamal_description/mesh/logos_maxi_base.stl" scale="0.001 0.001 0.001"/>
       </geometry>
       </collision>
@@ -50,5 +50,5 @@
       <geometry>
         <mesh
-          filename="package://hamal_description/mesh/wheel.stl" />
+          filename="package://hamal_description/mesh/wheel.stl" scale="0.001 0.001 0.001"/>
       </geometry>
       <material
@@ -80,5 +80,5 @@
       <geometry>
         <mesh
-          filename="package://hamal_description/mesh/wheel.stl" />
+          filename="package://hamal_description/mesh/wheel.stl" scale="0.001 0.001 0.001"/>
       </geometry>
       <material
@@ -90,8 +90,9 @@
     name="right_wheel_joint"
     type="continuous">
-      <origin
+      <!-- <origin
       xyz="0 -0.225 0.1"
-      rpy="0 0 0" />
-    <parent
+      rpy="0 0 0" /> -->
+      <origin xyz="0.1769 0 0" rpy="0 3.14 0" />
+      <parent
       link="base_link" />
     <child
@@ -104,5 +105,5 @@
   <link
     name="lifter_link">
-    <visual>
+    <!-- <visual>
       <origin
         xyz="0 0 0"
@@ -110,10 +111,10 @@
       <geometry>
         <mesh
-          filename="package://hamal_description/mesh/wheel.stl" />
+          filename="package://hamal_description/mesh/wheel.stl" scale="0.001 0.001 0.001"/>
       </geometry>
       <material
         name="red">
       </material>
-    </visual>
+    </visual> -->
   </link>
   <joint
