Commit message: Removed base_footprint from the TF tree, added move_base commands in the X direction for the base_link frame via manual commands.

File: hamal_description/urdf/hamal.urdf.xacro (robot description, xacro)
@@ -1,4 +1,4 @@
 <?xml version="1.0"?>
-<robot name="moobot" xmlns:xacro="http://ros.org/wiki/xacro">
+<robot name="hamal" xmlns:xacro="http://ros.org/wiki/xacro">
   <!-- AGV Base -->
   <link name="base_link">
@@ -25,10 +25,10 @@
     </inertial>
   </link>
-  <link name="base_footprint" />
+  <!-- <link name="base_link" />
   <joint name="base_joint" type="fixed">
-    <parent link="base_footprint" />
+    <parent link="base_link" />
     <child link="base_link" />
     <origin xyz="0 0 0" rpy="0 0 0" />
-  </joint>
+  </joint> -->
   <!-- Rear Right Mid Wheel Joint  -->
   <joint name="right_wheel_joint" type="continuous">

File: hamal_description/urdf/hamal_simple.urdf.xacro (robot description, xacro)
@@ -29,5 +29,5 @@
   </link>
     <!--link
-    name="base_footprint">
+    name="base_link">
   </link>
     <joint
@@ -38,5 +38,5 @@
       rpy="0 0 0" />
     <parent
-      link="base_footprint" />
+      link="base_link" />
     <child
       link="base_link" />

File: hamal_description/urdf/moobot.urdf.xacro (robot description, xacro)
@@ -27,7 +27,7 @@
     </inertial>
   </link>
-  <link name="base_footprint" />
+  <link name="base_link" />
   <joint name="base_joint" type="fixed">
-    <parent link="base_footprint" />
+    <parent link="base_link" />
     <child link="base_link" />
     <origin xyz="0 0 0" rpy="0 0 0" />

Commit message: Changed startup and control launch files.

File: hamal_description/urdf/hamal.urdf.xacro (robot description, xacro)
@@ -149,3 +149,16 @@
   </joint>
   <link name="imu_link"></link>
+  <joint name="camera_joint" type="fixed">
+    <parent link="base_link" />
+    <child link="camera_link" />
+    <origin xyz="0.80612 0.0 0.185" rpy="0 0 0" />
+  </joint>
+  <link name="camera_link">
+    <visual>
+      <origin xyz="0 0 0" rpy="0 0 0" />
+      <geometry>
+        <mesh filename="package://hamal_description/mesh/nanoscan.stl" scale="0.001 0.001 0.001" />
+      </geometry>
+    </visual>
+  </link>
 </robot>
